File: hardware/electronics/pcb.sch (KiCad schematic (older format))
At the start: 20 parts, among them IC1 23LC1024, M1 TSR1-2450, M2 TSR1-2433, P1 CONN_01X02, SW3 SWITCH_PUSHBUTTON, U1 74LS125, U2 74LS125

Commit message: New borad layout - routing incomplete
Parts:
- renumbered B1 to B?, C4 to C?, C3 to C?, C2 to C?, C1 to C?, C6 to C?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
