File: hardware/electronics/irm_pcb/Control.sch (KiCad schematic (older format))
At the start: 5 parts, among them J14 Conn_01x10, U3 74LS125, U4 74LS125

Commit message: New borad layout - routing incomplete
Parts:
- RV1: footprint irm_pcb:Potentiometer_Trimmer_Bourns_3339H_Horizontal -> irm_pcb:Potentiometer_Trimmer_Bourns_3386F
Changed lines of the file:
@@
 F 0 "RV1" V 6825 3150 50  0000 C CNN
 F 1 "10K" V 6900 3150 50  0000 C CNN
-F 2 "irm_pcb:Potentiometer_Trimmer_Bourns_3339H_Horizontal" H 7000 3150 50  0001 C CNN
+F 2 "irm_pcb:Potentiometer_Trimmer_Bourns_3386F" H 7000 3150 50  0001 C CNN
 F 3 "" H 7000 3150 50  0000 C CNN
 	1    7000 3150
