File: hardware/electronics/irm_pcb/MP3Codec.sch (KiCad schematic (older format))
At the start: 44 parts, among them J10 Conn_02x05_Counter_Clockwise, J11 Conn_01x04, J12 Conn_01x06, J13 Conn_01x06, J2 JUMPER_OPEN, J3 JUMPER_CLOSED, J4 JUMPER_CLOSED, J5 AudioJack3_Switch, J6 Screw_Terminal_1x02, J7 Screw_Terminal_1x02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

Commit message: New borad layout - routing incomplete
Parts:
- removed R5: 100K, Resistors_SMD:R_0805_HandSoldering, symbol modular-internet-radio:R
Connections:
- wire segments 191 -> 188
Other:
- note removed: "SPI BOOT DISABLE"
Changed lines of the file:
@@
 F 3 "" H 7175 3850 50  0001 C CNN
 	1    7200 3850
-	-1   0    0    1
+	-1   0    0    -1
 $EndComp
 $Comp
@@
 	1    0    0    -1
 $EndComp
-Text Notes 4350 700  0    60   ~ 0
-SPI BOOT DISABLE
 Text Notes 4000 1350 0    60   ~ 0
 MIDI BOOT WHEN \nJUMPER CLOSED
-$Comp
-L modular-internet-radio:R R?
-U 1 1 5DD30D51
-P 5000 800
-AR Path="/5DD30D51" Ref="R?"  Part="1"
-AR Path="/5DCC2CF1/5DD30D51" Ref="R5"  Part="1"
-F 0 "R5" V 5080 800 50  0000 C CNN
-F 1 "100K" V 5000 800 50  0000 C CNN
-F 2 "Resistors_SMD:R_0805_HandSoldering" V 4930 800 50  0001 C CNN
-F 3 "" H 5000 800 50  0000 C CNN
-	1    5000 800
-	0    1    1    0
-$EndComp
 $Comp
 L modular-internet-radio:R R?
@@
 	0    1    1    0
 $EndComp
-Text Label 4550 800  0    60   ~ 0
-GPIO0
 Text Label 4550 1050 0    60   ~ 0
 GPIO1
@@
 Connection ~ 3650 4000
 Wire Wire Line
-	4500 800  4850 800
-Wire Wire Line
 	4850 1050 4500 1050
 Wire Wire Line
@@
 Wire Wire Line
 	5150 1050 5250 1050
-Wire Wire Line
-	5150 800  5250 800
-Wire Wire Line
-	5250 800  5250 1050
 Wire Wire Line
 	4600 3900 4600 4000
@@
 SCK
 Connection ~ 1650 2700
-Connection ~ 5250 1050
 $Comp
 L modular-internet-radio:AGND #PWR?
